Commit message: Integrated IMU with robot_localization package for improved state estimation

File: description/gazebo_control.xacro (robot description, xacro)
@@ -6,5 +6,5 @@
             <left_joint>left_wheel_joint</left_joint>
             <right_joint>right_wheel_joint</right_joint>
-            <wheel_separation>0.35</wheel_separation>
+            <wheel_separation>0.2</wheel_separation>
             <wheel_diameter>0.1</wheel_diameter>
             <!-- Limits -->

File: description/lidar.xacro (robot description, xacro)
@@ -4,5 +4,5 @@
         <parent link="chassis"/>
         <child link="laser_frame"/>
-        <origin xyz="0.1 0 0.175" rpy="0 0 0"/>
+        <origin xyz="0.1 0 0.1" rpy="0 0 0"/>
     </joint>
     <link name="laser_frame">
@@ -51,3 +51,133 @@
         </sensor>
     </gazebo>
+    <!--IMU Sensor-->
+    <!--<joint name="imu_joint" type="fixed">
+        <parent link="chassis"/>
+        <child link="imu_link"/>
+        <origin xyz="0.2 0 0.1" rpy="0 0 0"/>
+    </joint>
+    <link name="imu_link">
+        <visual>
+            <geometry>
+                <box size="0.05 0.05 0.01"/>
+            </geometry>
+            <material name="white"/>
+        </visual>
+        <collision>
+            <geometry>
+                <box size="0.05 0.05 0.01"/>
+            </geometry>
+        </collision>
+        <xacro:inertial_box mass="0.01" x="0.2" y="0" z="0.1" >
+            <origin xyz="0.2 0 0.1" rpy="0 0 0"/>
+        </xacro:inertial_box>
+    </link>
+    <gazebo reference="imu_link">
+        <gravity>true</gravity>
+        <sensor name="imu_sensor" type="imu">
+          <always_on>true</always_on>
+          <update_rate>100</update_rate>
+          <visualize>true</visualize>
+          <topic>__default_topic__</topic>
+          <plugin filename="libgazebo_ros_imu_sensor.so" name="imu_plugin">
+            <topicName>imu</topicName>
+            <bodyName>imu_link</bodyName>
+            <updateRateHZ>10.0</updateRateHZ>
+            <gaussianNoise>0.0</gaussianNoise>
+            <xyzOffset>0 0 0</xyzOffset>
+            <rpyOffset>0 0 0</rpyOffset>
+            <frameName>imu_link</frameName>
+            <initialOrientationAsReference>false</initialOrientationAsReference>
+          </plugin>
+          <pose>0 0 0 0 0 0</pose>
+        </sensor>
+      </gazebo>-->
+    <link name="imu_link">
+        <visual>
+            <geometry>
+            <box size="0.05 0.05 0.01"/>
+            </geometry>
+        </visual>
+        <collision>
+            <geometry>
+            <box size="0.05 0.05 0.01"/>
+            </geometry>
+        </collision>
+        <xacro:inertial_box mass="0.01" x="0.05" y="0.05" z="0.01">
+            <origin xyz="0.1 0 0.1" rpy="0 0 0"/>
+        </xacro:inertial_box>
+    </link>
+    <joint name="imu_joint" type="fixed">
+        <parent link="base_link"/>
+        <child link="imu_link"/>
+        <origin xyz="0.1 0 0.1"/>
+    </joint>
+    <gazebo reference="imu_link">
+        <sensor name="imu_sensor" type="imu">
+            <plugin filename="libgazebo_ros_imu_sensor.so" name="imu_plugin">
+                <ros>
+                    <namespace>/demo</namespace>
+                    <remapping>~/out:=imu</remapping>
+                </ros>
+                <initial_orientation_as_reference>false</initial_orientation_as_reference>
+            </plugin>
+            <always_on>true</always_on>
+            <update_rate>100</update_rate>
+            <visualize>true</visualize>
+            <imu>
+                <angular_velocity>
+                    <x>
+                        <noise type="gaussian">
+                            <mean>0.0</mean>
+                            <stddev>2e-4</stddev>
+                            <bias_mean>0.0000075</bias_mean>
+                            <bias_stddev>0.0000008</bias_stddev>
+                        </noise>
+                    </x>
+                    <y>
+                        <noise type="gaussian">
+                            <mean>0.0</mean>
+                            <stddev>2e-4</stddev>
+                            <bias_mean>0.0000075</bias_mean>
+                            <bias_stddev>0.0000008</bias_stddev>
+                        </noise>
+                    </y>
+                    <z>
+                        <noise type="gaussian">
+                            <mean>0.0</mean>
+                            <stddev>2e-4</stddev>
+                            <bias_mean>0.0000075</bias_mean>
+                            <bias_stddev>0.0000008</bias_stddev>
+                        </noise>
+                    </z>
+                </angular_velocity>
+                <linear_acceleration>
+                    <x>
+                        <noise type="gaussian">
+                            <mean>0.0</mean>
+                            <stddev>1.7e-2</stddev>
+                            <bias_mean>0.1</bias_mean>
+                            <bias_stddev>0.001</bias_stddev>
+                        </noise>
+                    </x>
+                    <y>
+                        <noise type="gaussian">
+                            <mean>0.0</mean>
+                            <stddev>1.7e-2</stddev>
+                            <bias_mean>0.1</bias_mean>
+                            <bias_stddev>0.001</bias_stddev>
+                        </noise>
+                    </y>
+                    <z>
+                        <noise type="gaussian">
+                            <mean>0.0</mean>
+                            <stddev>1.7e-2</stddev>
+                            <bias_mean>0.1</bias_mean>
+                            <bias_stddev>0.001</bias_stddev>
+                        </noise>
+                    </z>
+                </linear_acceleration>
+            </imu>
+        </sensor>
+    </gazebo>
 </robot>

File: description/robot_core.xacro (robot description, xacro)
@@ -20,26 +20,33 @@
     <link name="base_link">
     </link>
+    <joint name="base_footprint_joint" type="fixed">
+        <parent link="base_link"/>
+        <child link="base_footprint"/>
+        <origin xyz="0 0 0" rpy="0 0 0"/>
+    </joint>
+    <link name="base_footprint">
+    </link>
     <!--CHASSIS LINK-->
     <joint name="chassis_joint" type="fixed">
         <parent link="base_link"/>
         <child link="chassis"/>
-        <origin xyz="-0.1 0 0"/>
+        <origin xyz="-0.125 0 0"/>
     </joint>
     <link name="chassis">
         <visual>
-            <origin xyz="0.15 0 0.075"/>
+            <origin xyz="0.125 0 0.05"/>
             <geometry>
-                <box size="0.3 0.3 0.15"/>
+                <box size="0.25 0.2 0.1"/>
             </geometry>
             <material name="white"/>
         </visual>
         <collision>
-            <origin xyz="0.15 0 0.075"/>
+            <origin xyz="0.125 0 0.05"/>
             <geometry>
-                <box size="0.3 0.3 0.15"/>
+                <box size="0.25 0.2 0.1"/>
             </geometry>
         </collision>
-        <xacro:inertial_box mass="0.5" x="0.3" y="0.3" z="0.15" >
-            <origin xyz="0.15 0 0.075" rpy="0 0 0"/>
+        <xacro:inertial_box mass="0.5" x="0.25" y="0.2" z="0.1" >
+            <origin xyz="0.125 0 0.05" rpy="0 0 0"/>
         </xacro:inertial_box>
     </link>
@@ -51,5 +58,5 @@
         <parent link="base_link"/>
         <child link="left_wheel"/>
-        <origin xyz="0 0.175 0" rpy="-${pi/2} 0 0"/>
+        <origin xyz="-0.0625 0.11 0" rpy="-${pi/2} 0 0"/>
         <axis xyz="0 0 1"/>
     </joint>
@@ -57,5 +64,5 @@
         <visual>
             <geometry>
-                <cylinder radius="0.05" length="0.04"/>
+                <cylinder radius="0.05" length="0.02"/>
             </geometry>
             <material name="blue"/>
@@ -63,8 +70,8 @@
         <collision>
             <geometry>
-                <cylinder radius="0.05" length="0.04"/>
+                <cylinder radius="0.05" length="0.02"/>
             </geometry>
         </collision>
-        <xacro:inertial_cylinder mass="0.1" length="0.04" radius="0.05">
+        <xacro:inertial_cylinder mass="0.1" length="0.02" radius="0.05">
             <origin xyz="0 0 0" rpy="0 0 0"/>
         </xacro:inertial_cylinder>
@@ -77,5 +84,5 @@
         <parent link="base_link"/>
         <child link="right_wheel"/>
-        <origin xyz="0 -0.175 0" rpy="${pi/2} 0 0"/>
+        <origin xyz="-0.0625 -0.11 0" rpy="${pi/2} 0 0"/>
         <axis xyz="0 0 -1"/>
     </joint>
@@ -83,5 +90,5 @@
         <visual>
             <geometry>
-                <cylinder radius="0.05" length="0.04"/>
+                <cylinder radius="0.05" length="0.02"/>
             </geometry>
             <material name="blue"/>
@@ -89,8 +96,8 @@
         <collision>
             <geometry>
-                <cylinder radius="0.05" length="0.04"/>
+                <cylinder radius="0.05" length="0.02"/>
             </geometry>
         </collision>
-        <xacro:inertial_cylinder mass="0.1" length="0.04" radius="0.05">
+        <xacro:inertial_cylinder mass="0.1" length="0.02" radius="0.05">
             <origin xyz="0 0 0" rpy="0 0 0"/>
         </xacro:inertial_cylinder>
@@ -101,7 +108,8 @@
     <!-- CASTER WHEEL LINK -->
     <joint name="caster_wheel_joint" type="fixed">
-        <parent link="chassis"/>
+        <parent link="base_link"/>
         <child link="caster_wheel"/>
-        <origin xyz="0.24 0 0"/>
+        <origin xyz="0.0625 0. 0" rpy="0 0 0"/>
+        <axis xyz="0 0 1"/>
     </joint>
     <link name="caster_wheel">
@@ -126,3 +134,57 @@
         <mu2 value="0.001"/>
     </gazebo>
+    <!--<joint name="follower_left_wheel_joint" type="fixed">
+        <parent link="base_link"/>
+        <child link="follower_left_wheel"/>
+        <origin xyz="0.0625 0.11 0" rpy="-${pi/2} 0 0"/>
+        <axis xyz="0 0 1"/>
+    </joint>
+    <link name="follower_left_wheel">
+        <visual>
+            <geometry>
+                <cylinder radius="0.05" length="0.02"/>
+            </geometry>
+            <material name="black"/>
+        </visual>
+        <collision>
+            <geometry>
+                <cylinder radius="0.05" length="0.02"/>
+            </geometry>
+        </collision>
+        <xacro:inertial_cylinder mass="0.1" length="0.02" radius="0.05">
+            <origin xyz="0 0 0" rpy="0 0 0"/>
+        </xacro:inertial_cylinder>
+    </link>
+    <gazebo reference="follower_left_wheel">
+        <material>Gazebo/Black</material>
+        <mu1 value="0.001"/>
+        <mu2 value="0.001"/>
+    </gazebo>
+    <<joint name="follower_right_wheel_joint" type="fixed">
+        <parent link="base_link"/>
+        <child link="follower_right_wheel"/>
+        <origin xyz="0.0625 -0.11 0" rpy="${pi/2} 0 0"/>
+        <axis xyz="0 0 -1"/>
+    </joint>
+    <link name="follower_right_wheel">
+        <visual>
+            <geometry>
+                <cylinder radius="0.05" length="0.02"/>
+            </geometry>
+            <material name="black"/>
+        </visual>
+        <collision>
+            <geometry>
+                <cylinder radius="0.05" length="0.02"/>
+            </geometry>
+        </collision>
+        <xacro:inertial_cylinder mass="0.1" length="0.02" radius="0.05">
+            <origin xyz="0 0 0" rpy="0 0 0"/>
+        </xacro:inertial_cylinder>
+    </link>
+    <gazebo reference="follower_right_wheel">
+        <material>Gazebo/Black</material>
+        <mu1 value="0.001"/>
+        <mu2 value="0.001"/>
+    </gazebo>-->
 </robot>

Commit message: configured diff_drive plugin for 4 wheels

File: description/gazebo_control.xacro (robot description, xacro)
@@ -2,14 +2,27 @@
 <robot xmlns:xacro="http://www.ros.org/wiki/xacro"  name="robot">
     <gazebo>
-        <plugin name="diff_drive" filename="libgazebo_ros_diff_drive.so">
-            <!-- WHEEL INFORMATION-->
+        <!--<plugin name="diff_drive" filename="libgazebo_ros_diff_drive.so">
+            <! WHEEL INFORMATION->
             <left_joint>left_wheel_joint</left_joint>
             <right_joint>right_wheel_joint</right_joint>
             <wheel_separation>0.2</wheel_separation>
             <wheel_diameter>0.1</wheel_diameter>
-            <!-- Limits -->
+            <Limits >
             <max_wheel_torque>200</max_wheel_torque>
             <max_wheel_acceleration>10.0</max_wheel_acceleration>
-            <!-- Output -->
+            < Output >
+            <odometry_frame>odom</odometry_frame>
+            <robot_base_frame>base_link</robot_base_frame>
+            <publish_odom>true</publish_odom>
+            <publish_odom_tf>true</publish_odom_tf>
+            <publish_wheel_tf>true</publish_wheel_tf>
+        </plugin>-->
+        <plugin name="skid_steer" filename="libgazebo_ros_skid_steer_drive.so">
+            <left_front_joint>left_front</left_front_joint>
+            <right_front_joint>right_front</right_front_joint>
+            <left_rear_joint>left_rear</left_rear_joint>
+            <right_rear_joint>right_rear</right_rear_joint>
+            <max_wheel_torque>200</max_wheel_torque>
+            <max_wheel_acceleration>10.0</max_wheel_acceleration>
             <odometry_frame>odom</odometry_frame>
             <robot_base_frame>base_link</robot_base_frame>

File: description/lidar.xacro (robot description, xacro)
@@ -93,4 +93,9 @@
         </sensor>
       </gazebo>-->
+      <joint name="imu_joint" type="fixed">
+        <parent link="base_link"/>
+        <child link="imu_link"/>
+        <origin xyz="0.1 0 0.1"/>
+    </joint>
     <link name="imu_link">
         <visual>
@@ -108,9 +113,4 @@
         </xacro:inertial_box>
     </link>
-    <joint name="imu_joint" type="fixed">
-        <parent link="base_link"/>
-        <child link="imu_link"/>
-        <origin xyz="0.1 0 0.1"/>
-    </joint>
     <gazebo reference="imu_link">
         <sensor name="imu_sensor" type="imu">

File: description/robot_core copy.xacro (robot description, xacro)
@@ -55,11 +55,11 @@
     </gazebo>
     <!--LEFT WHEEL LINK-->
-    <joint name="left_front" type="continuous">
+    <joint name="left_wheel_joint" type="continuous">
         <parent link="base_link"/>
-        <child link="left_wheel_front"/>
+        <child link="left_wheel"/>
         <origin xyz="-0.0625 0.11 0" rpy="-${pi/2} 0 0"/>
         <axis xyz="0 0 1"/>
     </joint>
-    <link name="left_wheel_front">
+    <link name="left_wheel">
         <visual>
             <geometry>
@@ -77,15 +77,15 @@
         </xacro:inertial_cylinder>
     </link>
-    <gazebo reference="left_wheel_front">
+    <gazebo reference="left_wheel">
         <material>Gazebo/Blue</material>
     </gazebo>
     <!--RIGHT WHEEL LINK-->
-    <joint name="right_front" type="continuous">
+    <joint name="right_wheel_joint" type="continuous">
         <parent link="base_link"/>
-        <child link="right_wheel_front"/>
+        <child link="right_wheel"/>
         <origin xyz="-0.0625 -0.11 0" rpy="${pi/2} 0 0"/>
         <axis xyz="0 0 -1"/>
     </joint>
-    <link name="right_wheel_front">
+    <link name="right_wheel">
         <visual>
             <geometry>
@@ -103,14 +103,42 @@
         </xacro:inertial_cylinder>
     </link>
-    <gazebo reference="right_wheel_front">
+    <gazebo reference="right_wheel">
         <material>Gazebo/Blue</material>
     </gazebo>
-    <joint name="left_rear" type="continuous">
+    <!-- CASTER WHEEL LINK -->
+    <joint name="caster_wheel_joint" type="fixed">
         <parent link="base_link"/>
-        <child link="left_wheel_rear"/>
+        <child link="caster_wheel"/>
+        <origin xyz="0.0625 0. 0" rpy="0 0 0"/>
+        <axis xyz="0 0 1"/>
+    </joint>
+    <link name="caster_wheel">
+        <visual>
+            <geometry>
+                <sphere radius="0.05"/>
+            </geometry>
+            <material name="black"/>
+        </visual>
+        <collision>
+            <geometry>
+                <sphere radius="0.05"/>
+            </geometry>
+        </collision>
+        <xacro:inertial_sphere mass="0.1" radius="0.05">
+            <origin xyz="0 0 0" rpy="0 0 0"/>
+        </xacro:inertial_sphere>
+    </link>
+    <gazebo reference="caster_wheel">
+        <material>Gazebo/Black</material>
+        <mu1 value="0.001"/>
+        <mu2 value="0.001"/>
+    </gazebo>
+    <!--<joint name="follower_left_wheel_joint" type="fixed">
+        <parent link="base_link"/>
+        <child link="follower_left_wheel"/>
         <origin xyz="0.0625 0.11 0" rpy="-${pi/2} 0 0"/>
         <axis xyz="0 0 1"/>
     </joint>
-    <link name="left_wheel_rear">
+    <link name="follower_left_wheel">
         <visual>
             <geometry>
@@ -128,15 +156,16 @@
         </xacro:inertial_cylinder>
     </link>
-    <gazebo reference="left_wheel_rear">
+    <gazebo reference="follower_left_wheel">
         <material>Gazebo/Black</material>
+        <mu1 value="0.001"/>
+        <mu2 value="0.001"/>
     </gazebo>
-    <!--RIGHT REAR WHEEL-->
-    <joint name="right_rear" type="continuous">
+    <<joint name="follower_right_wheel_joint" type="fixed">
         <parent link="base_link"/>
-        <child link="right_wheel_rear"/>
+        <child link="follower_right_wheel"/>
         <origin xyz="0.0625 -0.11 0" rpy="${pi/2} 0 0"/>
         <axis xyz="0 0 -1"/>
     </joint>
-    <link name="right_wheel_rear">
+    <link name="follower_right_wheel">
         <visual>
             <geometry>
@@ -154,6 +183,8 @@
         </xacro:inertial_cylinder>
     </link>
-    <gazebo reference="right_wheel_rear">
+    <gazebo reference="follower_right_wheel">
         <material>Gazebo/Black</material>
-    </gazebo>
+        <mu1 value="0.001"/>
+        <mu2 value="0.001"/>
+    </gazebo>-->
 </robot>

File: description/ros2_control copy.xacro (robot description, xacro)
@@ -5,5 +5,5 @@
             <plugin>gazebo_ros2_control/GazeboSystem</plugin>
         </hardware>
-        <joint name="left_front">
+        <joint name="left_wheel_joint">
             <command_interface name="velocity">
                 <param name="min">-10</param>
@@ -13,21 +13,5 @@
             <state_interface name="position"/>
         </joint>
-        <joint name="right_front">
-            <command_interface name="velocity">
-                <param name="min">-10</param>
-                <param name="min">10</param>
-            </command_interface>
-            <state_interface name="velocity"/>
-            <state_interface name="position"/>
-        </joint>
-        <joint name="left_rear">
-            <command_interface name="velocity">
-                <param name="min">-10</param>
-                <param name="min">10</param>
-            </command_interface>
-            <state_interface name="velocity"/>
-            <state_interface name="position"/>
-        </joint>
-        <joint name="right_rear">
+        <joint name="right_wheel_joint">
             <command_interface name="velocity">
                 <param name="min">-10</param>
